Commit message: refactor: Updated link/joint naming styles

File: DSFE_App/DSFE_Engine/assets/rigidbody_models/vispa/vispa.urdf (robot description, URDF)
Before this commit: robot VISPA, 7 links, 6 joints
Links:
- removed link Link_0
- removed link Link_1
- removed link Link_2
- removed link Link_3
- removed link Link_4
- removed link Link_5
- removed link Link_6
- added link link00, mass 0.627; visual mesh filename=package://vispa/meshes/Link0-DHReference-PublicRelease.stl
- added link link01, mass 2.328; visual mesh filename=package://vispa/meshes/Link1-DHReference-PublicRelease.stl
- added link link02, mass 3.995; visual mesh filename=package://vispa/meshes/Link2-DHReference-PublicRelease.stl
- added link link03, mass 2.328; visual mesh filename=package://vispa/meshes/Link3-DHReference-PublicRelease.stl
- added link link04, mass 3.157; visual mesh filename=package://vispa/meshes/Link4-DHReference-PublicRelease.stl
- added link link05, mass 2.695; visual mesh filename=package://vispa/meshes/Link5-DHReference-PublicRelease.stl
- added link link06, mass 0.924; visual mesh filename=package://vispa/meshes/Link6-DHReference-PublicRelease.stl
Joints:
- removed joint Joint_1
- removed joint Joint_2
- removed joint Joint_3
- removed joint Joint_4
- removed joint Joint_5
- removed joint Joint_6
- added joint joint01: type revolute, parent link00, child link01, origin xyz=0 0 0.18 rpy=0 0 0, axis 0 0 1, limit lower=-3.14149265359 upper=3.14149265359 effort=50 velocity=0.09395689
- added joint joint02: type revolute, parent link01, child link02, origin xyz=0 0 0 rpy=1.57079632679 -1.57079632679 0, axis 0 0 1, limit lower=-3.14149265359 upper=3.14149265359 effort=50 velocity=0.09395689
- added joint joint03: type revolute, parent link02, child link03, origin xyz=0.8 0 0 rpy=0 0 -1.57079632679, axis 0 0 1, limit lower=-3.14149265359 upper=3.14149265359 effort=50 velocity=0.09395689
- added joint joint04: type revolute, parent link03, child link04, origin xyz=0 0.65 0 rpy=-1.57079632679 0 0, axis 0 0 1, limit lower=-3.14149265359 upper=3.14149265359 effort=50 velocity=0.09395689
- added joint joint05: type revolute, parent link04, child link05, origin xyz=0 0 0 rpy=1.57079632679 0 0, axis 0 0 1, limit lower=-3.14149265359 upper=3.14149265359 effort=50 velocity=0.09395689
- added joint joint06: type revolute, parent link05, child link06, origin xyz=0 0.325 0 rpy=-1.57079632679 0 0, axis 0 0 1, limit lower=-3.14149265359 upper=3.14149265359 effort=50 velocity=0.09395689

Commit message: chore: Separate collision and mesh files for the VISPA

File: DSFE_App/DSFE_Engine/assets/rigidbody_models/vispa/vispa.urdf (robot description, URDF)
Before this commit: robot VISPA, 7 links, 6 joints
Links:
- link link00: geometry collision mesh filename=package://vispa/meshes/collision/link0_collision.stl; visual mesh filename=package://vispa/meshes/visual/Link0-DHReference-PublicRelea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
- link link01: geometry collision mesh filename=package://vispa/meshes/collision/link1_collision.stl; visual mesh filename=package://vispa/meshes/visual/Link1-DHReference-PublicRelea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
- link link02: geometry collision mesh filename=package://vispa/meshes/collision/link2_collision.stl; visual mesh filename=package://vispa/meshes/visual/Link2-DHReference-PublicRelea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
- link link03: geometry collision mesh filename=package://vispa/meshes/collision/link3_collision.stl; visual mesh filename=package://vispa/meshes/visual/Link3-DHReference-PublicRelea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
- link link04: geometry collision mesh filename=package://vispa/meshes/collision/link4_collision.stl; visual mesh filename=package://vispa/meshes/visual/Link4-DHReference-PublicRelea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
- link link05: geometry collision mesh filename=package://vispa/meshes/collision/link5_collision.stl; visual mesh filename=package://vispa/meshes/visual/Link5-DHReference-PublicRelea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
- link link06: geometry collision mesh filename=package://vispa/meshes/visual/Link6-DHReference-PublicRelea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; visual mesh filename=package://vispa/meshes/visual/Link6-DHReference-PublicRelea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
